File: AutonomousSeedDistributor.kicad_pcb (KiCad board)
At the start: 4 copper layers, 59 parts, among them J1 Antenna, J2 RJ45_Wuerth_7499010121A, Q1 SELECT PART, Q2 SELECT PART, Q3 SELECT PART, Q4 SELECT PART, Q5 SELECT PART, U5 AP2127K-1.8, Y1 25M

Commit message: done with my subsystem
Parts:
- moved C11 1.40 mm to (130.0, 66.7)
- moved R5 1.40 mm to (130.2, 70.5)
- moved C13 1.00 mm to (117.0, 56.5)
Connections:
- R6 pad 2: Net-(R6-Pad2) -> GND
- R7 pad 2: Net-(R6-Pad2) -> GND
Routing:
- net GND: track 7.63 -> 89.5 mm, vias 0 -> 30
- net +3V3: track 10.7 -> 33.3 mm, vias 0 -> 11
- net VCCIO: track 14.0 -> 18.4 mm, vias 0 -> 6
- net Net-(J2-Pad10): track 2.56 -> 3.96 mm
- net Net-(J2-RCT): track 7.26 -> 8.66 mm
- net /Communication/LINK: track 20.2 -> 18.8 mm
- added copper zone on In2.Cu, net +3V3
- added copper zone on F.Cu, net GND
- added copper zone on In1.Cu, net GND
- added copper zone on F.Cu, net Net-(C13-Pad1)
- added copper zone on In2.Cu, net VCCIO

Commit message: combined, submitted for Packaging Review
Parts:
- added C22: C_Polarized, Capacitor_SMD:CP_Elec_4x3, F.Cu at (186.4, 109.6)
- added C23: C, Capacitor_SMD:C_0603_1608Metric, F.Cu at (191.4, 110.8)
- added C24: C_Polarized, Capacitor_SMD:CP_Elec_4x3, F.Cu at (175.4, 94.6)
- added C25: C, Capacitor_SMD:C_0603_1608Metric, F.Cu at (166.8, 119.0)
- added C26: C, Capacitor_SMD:C_0603_1608Metric, F.Cu at (192.6, 120.6)
- added D5: D, Diode_SMD:D_0603_1608Metric, F.Cu at (192.2, 107.8)
- added D6: SS38, Diode_SMD:D_SMA, F.Cu at (181.2, 105.2)
- added J3: Screw_Terminal_01x02, TerminalBlock:TerminalBlock_Xinya_XY308-2.54-2P_1x02_P2.54mm_Horizontal, F.Cu at (199.3, 105.1)
- added J4: Screw_Terminal_01x02, TerminalBlock:TerminalBlock_Xinya_XY308-2.54-2P_1x02_P2.54mm_Horizontal, F.Cu at (199.1, 129.5)
- added J5: Screw_Terminal_01x02, TerminalBlock:TerminalBlock_Xinya_XY308-2.54-2P_1x02_P2.54mm_Horizontal, F.Cu at (199.3, 97.3)
- added J6: Screw_Terminal_01x02, TerminalBlock:TerminalBlock_Xinya_XY308-2.54-2P_1x02_P2.54mm_Horizontal, F.Cu at (199.0, 117.3)
- added L2: L, Inductor_SMD:L_Chilisin_BMRA00050530, F.Cu at (181.2, 99.8)
- added L3: L, Inductor_SMD:L_SXN_SMDRI73, F.Cu at (173.0, 118.2)
- added M1: Motor_DC, Connector_PinHeader_1.27mm:PinHeader_1x02_P1.27mm_Vertical, F.Cu at (123.4, 115.2)
- added M2: Motor_DC, Connector_PinHeader_1.27mm:PinHeader_1x02_P1.27mm_Vertical, F.Cu at (123.2, 129.8)
- added M3: Motor_Servo, Connector_PinHeader_2.54mm:PinHeader_1x03_P2.54mm_Vertical, F.Cu at (157.9, 131.2)
- added M4: Motor_DC, Connector_PinHeader_1.27mm:PinHeader_1x02_P1.27mm_Vertical, F.Cu at (123.6, 103.0)
- added Q6: NMOS, Package_TO_SOT_SMD:Infineon_PG-HSOF-8-1, F.Cu at (134.5, 101.0)
- added R19: 100Ω, Resistor_SMD:R_0603_1608Metric, F.Cu at (160.2, 126.8)
- added R20: 100Ω, Resistor_SMD:R_0603_1608Metric, F.Cu at (131.2, 108.0)
- added R21: 100KΩ, Resistor_SMD:R_0603_1608Metric, F.Cu at (128.4, 108.8)
- added R22: 100kΩ, Resistor_SMD:R_0603_1608Metric, F.Cu at (188.2, 81.6)
- added R23: R_US, Resistor_SMD:R_0603_1608Metric, F.Cu at (179.6, 122.4)
- added R24: R_US, Resistor_SMD:R_0603_1608Metric, F.Cu at (179.6, 119.0)
- added U6: L298HN, Package_TO_SOT_THT:TO-220-15_P2.54x2.54mm_StaggerOdd_Lead5.84mm_TabDown, F.Cu at (128.8, 114.5)
- added U7: STM32F091CBTx, Package_QFP:LQFP-48_7x7mm_P0.5mm, F.Cu at (196.4, 80.6)
- added U8: LM2596S-3.3, Package_TO_SOT_SMD:TO-263-5_TabPin3, F.Cu at (166.8, 104.4)
- added VR1: TPS561208DDCR, Package_TO_SOT_SMD:TSOT-23-6_HandSoldering, F.Cu at (185.8, 120.8)
Connections:
- net GPIO_PC2 renamed B2
- net GPIO_PC3 renamed B8
- net SPI_MISO renamed SPI1_MISO
- net SPI_MOSI renamed SPI1_MOSI
- net SPI_SCK renamed SPI1_SCK
- U1 pad 31: GPIO_PC7 -> B7
- U1 pad 36: GPIO_PC4 -> B9
- U1 pad 59: GPIO_PC5 -> B12
- U1 pad 60: GPIO_PC6 -> B6
- U2 pad 4: GPIO_PC1 -> B1
Routing:
- net B13: track 0.00 -> 86.2 mm, vias 0 -> 2
- net UART4_RX: track 0.00 -> 85.3 mm, vias 0 -> 2
- net A7: track 0.00 -> 85.1 mm, vias 0 -> 1
- net A6: track 0.00 -> 83.2 mm, vias 0 -> 1
- net A5: track 0.00 -> 82.7 mm, vias 0 -> 1
- net A4: track 0.00 -> 81.0 mm, vias 0 -> 1
- net B12: track 0.00 -> 69.8 mm, vias 0 -> 2
- net B1: track 0.00 -> 69.7 mm, vias 0 -> 2
- net UART3_TX: track 0.00 -> 68.3 mm, vias 0 -> 2
- net B14: track 0.00 -> 67.5 mm, vias 0 -> 2
- net B6: track 0.00 -> 66.0 mm, vias 0 -> 2
- net UART3_RX: track 0.00 -> 64.9 mm, vias 0 -> 2
- net UART2_RX: track 0.00 -> 61.5 mm, vias 0 -> 2
- net UART4_TX: track 0.00 -> 60.0 mm, vias 0 -> 2
- net UART2_TX: track 0.00 -> 59.5 mm, vias 0 -> 2
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- added copper zone on In2.Cu, net +12V
- added copper zone on F.Cu, net +3V3
- added copper zone on In2.Cu, net +5V
Other:
- board outline added: 110 x 99 mm

Commit message: rev 1
Parts:
- removed D3, D4: LED, LED_SMD:LED_0603_1608Metric
- removed D5: D, Diode_SMD:D_0603_1608Metric
- removed D6: SS38, Diode_SMD:D_SMA
- removed JP1: SolderJumper_3_Open, Jumper:SolderJumper-3_P1.3mm_Open_RoundedPad1.0x1.5mm_NumberLabels
- removed L3: L, Inductor_SMD:L_SXN_SMDRI73
- removed M1, M2, M4: Motor_DC, Connector_PinHeader_1.27mm:PinHeader_1x02_P1.27mm_Vertical
- removed M3: Motor_Servo, Connector_PinHeader_2.54mm:PinHeader_1x03_P2.54mm_Vertical
- removed VR1: TPS561208DDCR, Package_TO_SOT_SMD:TSOT-23-6_HandSoldering
- added C27: 0.1uF, Capacitor_SMD:C_0603_1608Metric, F.Cu at (122.5, 88.0)
- added C28: 0.1uF, Capacitor_SMD:C_0603_1608Metric, F.Cu at (124.5, 92.2)
- added F1: MF-RHT1000, Fuse:Fuse_Bourns_MF-RHT1000, F.Cu at (124.0, 139.0)
- added H1: MountingHole, MountingHole:MountingHole_2.7mm, F.Cu at (84.0, 75.0)
- added H2: MountingHole, MountingHole:MountingHole_2.7mm, F.Cu at (142.0, 75.0)
- added H3: MountingHole, MountingHole:MountingHole_2.7mm, F.Cu at (84.0, 124.0)
- added H4: MountingHole, MountingHole:MountingHole_2.7mm, F.Cu at (142.0, 124.0)
- added J10: Conn_02x20_Odd_Even, Connector_PinSocket_2.54mm:PinSocket_2x20_P2.54mm_Vertical, B.Cu at (88.9, 76.3)
- added J11: Conn_01x04_Pin, Connector_PinHeader_2.54mm:PinHeader_1x04_P2.54mm_Vertical, F.Cu at (113.4, 81.5)
- added J12: Battery holes, 1984617(1):PHOENIX_1984617, F.Cu at (113.6, 142.3)
- added J13: USB_C_Receptacle, Connector_USB:USB_C_Receptacle_Amphenol_12401610E4-2A, F.Cu at (85.0, 85.0)
- added J7: Conn_01x03_Pin, Connector_PinHeader_2.54mm:PinHeader_1x03_P2.54mm_Vertical, F.Cu at (96.0, 89.8)
- added J8: Conn_01x04, Connector_PinHeader_2.54mm:PinHeader_1x04_P2.54mm_Vertical, F.Cu at (95.8, 102.5)
- added J9: Conn_01x02, 1984617(1):PHOENIX_1984617, F.Cu at (80.7, 105.8)
- added Q10: DMP3013SFV, Package_SON:Diodes_PowerDI3333-8, F.Cu at (100.5, 107.9)
- added Q11: BSS138, Package_TO_SOT_SMD:SOT-23, F.Cu at (100.2, 101.9)
- added Q7: BSS138, Package_TO_SOT_SMD:SOT-23, F.Cu at (106.3, 87.8)
- added Q8: BSS138, Package_TO_SOT_SMD:SOT-23, F.Cu at (102.0, 91.5)
- added Q9: BSS138, Package_TO_SOT_SMD:SOT-23, F.Cu at (104.0, 83.8)
- added R25: 4.7kR, Resistor_SMD:R_0603_1608Metric, F.Cu at (126.5, 119.2)
- added R26: 4.7kR, Resistor_SMD:R_0603_1608Metric, F.Cu at (126.5, 121.0)
- added R27: 20kR, Resistor_SMD:R_0603_1608Metric, F.Cu at (123.7, 113.1)
- added R28: 110kR, Resistor_SMD:R_0603_1608Metric, F.Cu at (121.2, 109.0)
- added R29: 15kR, Resistor_SMD:R_0603_1608Metric, F.Cu at (124.8, 109.0)
- added R30: 2.2kR, Resistor_SMD:R_0603_1608Metric, F.Cu at (137.2, 113.0)
- added R31: 5.1kR, Resistor_SMD:R_0603_1608Metric, F.Cu at (92.5, 85.0)
- added R32: 5.1kR, Resistor_SMD:R_0603_1608Metric, F.Cu at (85.0, 91.5)
- added U9: MIC5219-3.3YMM, Package_SO:MSOP-8_3x3mm_P0.65mm, F.Cu at (118.2, 91.0)
- C1, C15, C2, C21: value 0.1uF -> 1uF
- C10, C9: value ?? F -> 5pF
- C11: value 1uF -> 0.1uF; moved to F.Cu
- C12, C6: value 1uF -> 0.1uF
- C13: value 1nF -> 22uF
- C14: value 10uF -> 33nF
- C16: value 470pF -> 0.1uF
- C17: value 0.1uF -> 2.2nF
- C19, C20: value 1uF -> 47pF
- C22: value C_Polarized -> 60uF; footprint Capacitor_SMD:CP_Elec_4x3 -> Capacitor_SMD:C_0603_1608Metric
- C23, C25, C26: value C -> 0.1uF
- C24: value C_Polarized -> 0.1uF; footprint Capacitor_SMD:CP_Elec_4x3 -> Capacitor_SMD:C_0603_1608Metric
- C3: value 0.1uF -> 470pF
- C8: value 0.1uF -> 10uF
- D1: value LED -> 45V16A1; footprint LED_SMD:LED_0603_1608Metric -> Package_TO_SOT_THT:TO-220-2_Vertical
- D2: value LED -> 18VWM29.2VC1; footprint LED_SMD:LED_0603_1608Metric -> Diode_SMD:D_SOD-123
- J2: value RJ45_Wuerth_7499010121A -> Conn_01x04; footprint Connector_RJ:RJ45_Wuerth_7499010121A_Horizontal -> Connector_PinHeader_2.54mm:PinHeader_1x04_P2.54mm_Vertical
- J3, J6: value Screw_Terminal_01x02 -> Conn_01x04; footprint TerminalBlock:TerminalBlock_Xinya_XY308-2.54-2P_1x02_P2.54mm_Horizontal -> Connector_PinHeader_2.54mm:PinHeader_1x04_P2.54mm_Vertical
- J4, J5: value Screw_Terminal_01x02 -> Conn_01x06; footprint TerminalBlock:TerminalBlock_Xinya_XY308-2.54-2P_1x02_P2.54mm_Horizontal -> Connector_JST:JST_PH_B6B-PH-K_1x06_P2.00mm_Vertical
- L2: value L -> 4.7uH; footprint Inductor_SMD:L_Chilisin_BMRA00050530 -> 74437377047:WE-LHMI_1335
- Q1, Q2, Q3, Q4, Q5: value SELECT PART -> BSS138
- Q6: value NMOS -> BSS138; footprint Package_TO_SOT_SMD:Infineon_PG-HSOF-8-1 -> Package_TO_SOT_SMD:SOT-23
- R1: value 0R -> 10kR
- R10, R11, R12, R13, R14, R15, R16, R17, R8: value 2.2kR -> 10kR
- R18: value 2.2kR -> 100R
- R19: value 100Ω -> 10kR
- R2, R3, R4, R6, R7, R9: value 1kR -> 10kR
- R20: value 100Ω -> 50kR
- R21: value 100KΩ -> 100kR
- R22: value 100kΩ -> 10R
- R23: value R_US -> 7.5mR; footprint Resistor_SMD:R_0603_1608Metric -> Resistor_SMD:R_2512_6332Metric
- R24: value R_US -> 10R
- R5: value 1kR -> 10kR; moved to F.Cu
- U1: value ~ -> AP2127K-1.8; footprint Package_QFP:LQFP-64_10x10mm_P0.5mm -> Package_TO_SOT_SMD:SOT-23-5
- U2: footprint jshep:LCC-18 -> jshep:uDFN-6
- U4: footprint jshep:uDFN-6 -> jshep:LCC-18
- U5: value AP2127K-1.8 -> L298HN; footprint Package_TO_SOT_SMD:SOT-23-5 -> Package_TO_SOT_THT:TO-220-15_P2.54x2.54mm_StaggerOdd_Lead5.84mm_TabDown
- U6: value L298HN -> STM32F091RCT6; footprint Package_TO_SOT_THT:TO-220-15_P2.54x2.54mm_StaggerOdd_Lead5.84mm_TabDown -> Package_QFP:LQFP-64_10x10mm_P0.5mm
- U7: value STM32F091CBTx -> INA226AQDGSRQ1; footprint Package_QFP:LQFP-48_7x7mm_P0.5mm -> Package_SO:VSSOP-10_3x3mm_P0.5mm
- U8: value LM2596S-3.3 -> AOZ6605PI-1; footprint Package_TO_SOT_SMD:TO-263-5_TabPin3 -> AOZ6605PI-1:SO8_EP1_AOS
- Y1: value 25M -> CM7V-T1A-32.768kHz-7pF; footprint Crystal:Crystal_SMD_7050-4Pin_7.0x5.0mm -> Crystal:Crystal_SMD_3215-2Pin_3.2x1.5mm
- moved J5 123.9 mm to (83.0, 140.0), turned to 0 degrees
- moved J3 112.3 mm to (87.0, 102.6), turned to 180 degrees
- moved J6 108.7 mm to (91.2, 102.6), turned to 180 degrees
- moved J4 100.6 mm to (99.0, 140.0), turned to 0 degrees
- moved U2 97.9 mm to (129.8, 140.6), turned to 90 degrees
- moved J1 96.0 mm to (140.8, 141.0), turned to -90 degrees
- moved L1 94.6 mm to (133.2, 141.0), turned to 180 degrees
- moved R14 92.8 mm to (104.5, 95.0)
- moved U4 92.3 mm to (128.0, 137.1), turned to 90 degrees
- moved R18 89.8 mm to (99.0, 88.2), turned to -90 degrees
- moved R13 87.8 mm to (100.9, 83.8), turned to 90 degrees
- moved U7 85.2 mm to (121.5, 121.2), turned to 180 degrees
- moved U5 83.9 mm to (107.1, 113.0), turned to 180 degrees
- moved R12 83.6 mm to (99.1, 91.5), turned to 90 degrees
- moved R11 83.0 mm to (103.3, 87.8), turned to 90 degrees
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Connections:
- C1 pad 1: VCCIO -> GND
- C1 pad 2: GND -> +3V3
- C10 pad 2: /Communication/XO -> Net-(U6-PC15-OSC32_OUT)
- C11 pad 1: Net-(J2-RCT) -> Net-(C11-Pad1)
- C11 pad 2: GND -> Net-(U7-IN+)
- C12 pad 1: Net-(J2-TCT) -> Net-(U7-VS)
- C12 pad 2: GND -> +3V3
- C13 pad 1: Net-(C13-Pad1) -> VBAT_LOAD
- C14 pad 1: +3V3 -> GND
- C14 pad 2: GND -> Net-(U8-SS)
- C15 pad 1: GND -> +5V
- C15 pad 2: +3V3 -> GND
- C16 pad 1: Net-(C16-Pad1) -> Net-(U8-VCC)
- C16 pad 2: Net-(J1-In) -> GND
- C17 pad 1: GND -> Net-(C17-Pad1)
- C17 pad 2: +1V8 -> GND
- C18 pad 1: GND -> Net-(U8-LX)
- C18 pad 2: Net-(U3-REGOUT) -> Net-(U8-BST)
- C19 pad 1: GND -> Net-(U8-COMP)
- C19 pad 2: +1V8 -> GND
- C2 pad 1: VCCIO -> GND
- C2 pad 2: GND -> +1V8
- C20 pad 1: GND -> +5V
- C20 pad 2: +3V3 -> Net-(U8-FB)
- C21 pad 1: GND -> +3V3
- C21 pad 2: +1V8 -> GND
- C22 pad 1: Net-(D5-K) -> +5V
- C23 pad 1: Net-(D5-K) -> +3V3
- C25 pad 1: Net-(C25-Pad1) -> +3V3
- C26 pad 1: GND -> +3V3
- C26 pad 2: +12V -> GND
- C3 pad 1: VCCIO -> Net-(C3-Pad1)
- C3 pad 2: GND -> Net-(J1-In)
- C4 pad 1: VCCIO -> GND
- C4 pad 2: GND -> +1V8
- C5 pad 1: VCCIO -> GND
- C5 pad 2: GND -> +3V3
- C6 pad 1: Net-(C6-Pad1) -> GND
- C6 pad 2: GND -> Net-(U3-REGOUT)
- C7 pad 1: Net-(C7-Pad1) -> GND
- C7 pad 2: GND -> +1V8
- C8 pad 1: Net-(C8-Pad1) -> +3V3
- C9 pad 2: /Communication/XI -> Net-(U6-PC14-OSC32_IN)
- D1 pad 1: Net-(D1-K) -> VBAT
- D1 pad 2: /Communication/TCPCS1 -> Net-(D1-A)
- D2 pad 1: Net-(D2-K) -> VBAT
- D2 pad 2: /Communication/TCPCS2 -> GND
- J2 pad 1: /Communication/TXP -> +5V
- J2 pad 2: Net-(J2-TCT) -> US1_TRIG
- J2 pad 3: /Communication/TXN -> /Motor Control/ECHO1
- J2 pad 4: /Communication/RXP -> GND
- J3 pad 1: GND -> +5V
- J3 pad 2: +12V -> US2_TRIG
- J4 pad 1: GND -> /Motor Control/M1+
- J4 pad 2: +5V -> +3V3
- J5 pad 1: +3V3 -> /Motor Control/M2+
- J5 pad 2: GND -> +3V3
- J6 pad 1: GND -> +5V
- J6 pad 2: +12V -> US3_TRIG
- L1 pad 1: Net-(C16-Pad1) -> Net-(C3-Pad1)
- L1 pad 2: Net-(U4-RFIN) -> Net-(U2-RFIN)
- L2 pad 1: Net-(D6-K) -> Net-(U8-LX)
- L2 pad 2: +3V3 -> +5V
- Q1 pad 2: /Positioning/SDO -> /Positioning/nCS
- Q1 pad 3: SPI1_MISO -> IMU_nCS
- Q2 pad 3: B8 -> IMU_INT
- Q3 pad 2: /Positioning/nCS -> /Positioning/SDO
- Q3 pad 3: B2 -> SPI1_MISO
- Q6 pad 1: Net-(M4--) -> +5V
- Q6 pad 2: Net-(Q6-G) -> /Motor Control/ECHO4
- Q6 pad 3: GND -> US4_ECHO
- R1 pad 1: +3V3 -> /Positioning/nCS
- R1 pad 2: VCCIO -> +1V8
- R10 pad 1: SPI1_MISO -> /Motor Control/ECHO4
- R10 pad 2: +3V3 -> +5V
- R11 pad 1: /Positioning/INT1 -> /Motor Control/ECHO2
- R11 pad 2: +1V8 -> +5V
- R12 pad 1: B8 -> /Motor Control/ECHO3
- R12 pad 2: +3V3 -> +5V
- R13 pad 1: /Positioning/nCS -> /Motor Control/ECHO1
- R13 pad 2: +1V8 -> +5V
- R14 pad 1: B2 -> US4_ECHO
- R15 pad 1: /Positioning/SDI -> US2_ECHO
- R15 pad 2: +1V8 -> +3V3
- R16 pad 1: SPI1_MOSI -> US3_ECHO
- R17 pad 1: /Positioning/SCLK -> US1_ECHO
- R17 pad 2: +1V8 -> +3V3
- R18 pad 1: SPI1_SCK -> SERVO_PWM
- R18 pad 2: +3V3 -> Net-(J7-Pin_1)
- R19 pad 1: B14 -> Net-(Q11-D)
- R19 pad 2: Net-(M3-PWM) -> Net-(Q10-G)
- R2 pad 1: Net-(D1-K) -> /Positioning/INT1
- R2 pad 2: GND -> +1V8
- R20 pad 1: B13 -> VBAT_LOAD
- R20 pad 2: Net-(Q6-G) -> Net-(Q10-G)
- R21 pad 1: Net-(Q6-G) -> NRST
- R21 pad 2: GND -> +3V3
- R22 pad 1: +3V3 -> Net-(U7-IN-)
- R22 pad 2: Net-(U7-NRST) -> VBAT_LOAD
- R23 pad 1: +5V -> VBAT_LOAD
- R23 pad 2: Net-(VR1-VFB) -> VBAT
- R24 pad 1: Net-(VR1-VFB) -> Net-(C11-Pad1)
- R24 pad 2: Net-(L3-Pad2) -> VBAT
- R3 pad 1: Net-(D2-K) -> /Positioning/SDO
- R3 pad 2: GND -> +1V8
- R4 pad 1: /Communication/ACT -> /Positioning/SDI
- R4 pad 2: Net-(J2-Pad12) -> +1V8
- R5 pad 1: /Communication/LINK -> IMU_nCS
- R5 pad 2: Net-(J2-Pad10) -> +3V3
- R6 pad 1: Net-(D3-K) -> IMU_INT
- R6 pad 2: GND -> +3V3
- R7 pad 1: Net-(D4-K) -> SPI1_MISO
- R7 pad 2: GND -> +3V3
- R8 pad 1: /Positioning/SDO -> SPI1_MOSI
- R8 pad 2: +1V8 -> +3V3
- R9 pad 1: Net-(JP1-A) -> SPI1_SCK
- R9 pad 2: Net-(U1-CFGEN) -> +3V3
- U1 pad 1: unconnected-(U1-NC-Pad1) -> +3V3
- U1 pad 2: +3V3 -> GND
- U1 pad 3: GND -> +3V3
- U1 pad 4: /Communication/RXP -> unconnected-(U1-NC-Pad4)
- U1 pad 5: /Communication/RXN -> +1V8
- U2 pad 2: UART4_TX -> GND
- U2 pad 3: UART4_RX -> Net-(U2-RFIN)
- U2 pad 4: B1 -> +3V3
- U2 pad 5: unconnected-(U2-ON/OFF-Pad5) -> +3V3
- U2 pad 6: Net-(BT1-+) -> Net-(U2-RFOUT)
- U4 pad 2: GND -> UART2_TX
- U4 pad 3: Net-(U4-RFIN) -> UART2_RX
- U4 pad 4: +3V3 -> unconnected-(U4-1PPS-Pad4)
- U4 pad 5: +3V3 -> unconnected-(U4-ON/OFF-Pad5)
- U4 pad 6: Net-(U2-RF_IN) -> Net-(BT1-+)
- U5 pad 1: +3V3 -> GND
- U5 pad 2: GND -> /Motor Control/M1+
- U5 pad 3: +3V3 -> /Motor Control/M1-
- U5 pad 4: unconnected-(U5-NC-Pad4) -> VBAT_LOAD
- U5 pad 5: +1V8 -> M1_IN1_PWM
- U6 pad 1: GND -> +3V3
- U6 pad 10: A6 -> US3_TRIG
- U6 pad 11: +5V -> US4_TRIG
- U6 pad 12: A7 -> GND
- U6 pad 13: Net-(M2-+) -> +3V3
- U6 pad 14: Net-(M2--) -> M1_ENCA
- U6 pad 15: GND -> M1_ENCB
- U6 pad 2: Net-(M1-+) -> unconnected-(U6-PC13-Pad2)
- U6 pad 3: Net-(M1--) -> Net-(U6-PC14-OSC32_IN)
- U6 pad 4: +12V -> Net-(U6-PC15-OSC32_OUT)
- U6 pad 5: A4 -> I2C1_SDA
- U6 pad 6: +5V -> I2C1_SCK
- U6 pad 7: A5 -> NRST
- U6 pad 8: GND -> US1_TRIG
- U6 pad 9: +5V -> US2_TRIG
- U7 pad 1: +3V3 -> GND
- U7 pad 10: UART4_TX -> Net-(U7-IN+)
- U7 pad 2: C13 -> GND
- U7 pad 3: C14 -> unconnected-(U7-ALERT-Pad3)
- U7 pad 4: C15 -> I2C1_SDA
- U7 pad 5: F0 -> I2C1_SCK
- U7 pad 6: F1 -> Net-(U7-VS)
- U7 pad 7: Net-(U7-NRST) -> GND
- U7 pad 8: GND -> Net-(U7-IN-)
- U7 pad 9: +3V3 -> Net-(U7-IN-)
- U8 pad 1: Net-(D5-K) -> Net-(U8-SS)
- U8 pad 2: Net-(D6-K) -> VBAT_LOAD
- U8 pad 3: GND -> VBAT_LOAD
- U8 pad 4: +3V3 -> GND
- U8 pad 5: GND -> Net-(U8-BST)
- Y1 pad 1: /Communication/XO -> Net-(U6-PC15-OSC32_OUT)
- Y1 pad 2: GND -> Net-(U6-PC14-OSC32_IN)
Routing:
- net M2_ENCB: track 0.00 -> 107.0 mm, vias 0 -> 1
- net M2_ENCA: track 0.00 -> 105.4 mm, vias 0 -> 1
- net B13: track 86.2 -> 0.00 mm, vias 2 -> 0
- net UART4_RX: track 85.3 -> 0.00 mm, vias 2 -> 0
- net A7: track 85.1 -> 0.00 mm, vias 1 -> 0
- net M1_ENCB: track 0.00 -> 84.6 mm, vias 0 -> 1
- net M1_ENCA: track 0.00 -> 84.6 mm, vias 0 -> 1
- net A6: track 83.2 -> 0.00 mm, vias 1 -> 0
- net A5: track 82.7 -> 0.00 mm, vias 1 -> 0
- net A4: track 81.0 -> 0.00 mm, vias 1 -> 0
- net US1_TRIG: track 0.00 -> 74.4 mm, vias 0 -> 1
- net US2_TRIG: track 0.00 -> 70.6 mm, vias 0 -> 1
- net B12: track 69.8 -> 0.00 mm, vias 2 -> 0
- net B1: track 69.7 -> 0.00 mm, vias 2 -> 0
- net UART3_TX: track 68.3 -> 0.00 mm, vias 2 -> 0
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- added copper zone on F.Cu, net +5V
- added copper zone on F.Cu, net Net-(D1-A)
- added copper zone on F.Cu, net Net-(J12-Pin_2)
- added copper zone on F.Cu, net Net-(J9-Pin_1)
- added copper zone on F.Cu, net Net-(U8-LX)
- added copper zone on F.Cu, net VBAT
- added copper zone on F.Cu, net VBAT_LOAD
- added copper zone on In2.Cu, net VBAT_LOAD
- removed copper zone on In2.Cu, net +12V
- removed copper zone on F.Cu, net +1V8
- removed copper zone on F.Cu, net +3V3
- removed copper zone on F.Cu, net GND
- removed copper zone on F.Cu, net Net-(C13-Pad1)
- removed copper zone on In2.Cu, net VCCIO
Other:
- board size 110 x 99 mm -> 65 x 73 mm
- board text added: "+"
- board text added: "-"
