File: McuAndPower.kicad_sch (KiCad schematic)
At the start: 19 parts, among them J3 Screw_Terminal_01x02, J4 Screw_Terminal_01x02, J5 Screw_Terminal_01x02, J6 Screw_Terminal_01x02, U7 STM32F091CBTx, U8 LM2596S-3.3

Commit message: rev 1
Parts:
- removed C22, C24: C_Polarized, Capacitor_SMD:CP_Elec_4x3, symbol Device:C_Polarized
- removed C23, C25, C26: C, Capacitor_SMD:C_0603_1608Metric, symbol Device:C
- removed D5: D, Diode_SMD:D_0603_1608Metric, symbol Device:D
- removed D6: SS38, Diode_SMD:D_SMA, symbol Diode:SS38
- removed J3, J4, J5, J6: Screw_Terminal_01x02, TerminalBlock:TerminalBlock_Xinya_XY308-2.54-2P_1x02_P2.54mm_Horizontal, symbol Connector:Screw_Terminal_01x02
- removed L3: L, Inductor_SMD:L_SXN_SMDRI73, symbol Device:L
- removed R22: 100kΩ, Resistor_SMD:R_0603_1608Metric, symbol Device:R
- removed U7: STM32F091CBTx, Package_QFP:LQFP-48_7x7mm_P0.5mm, symbol MCU_ST_STM32F0:STM32F091CBTx
- removed U8: LM2596S-3.3, Package_TO_SOT_SMD:TO-263-5_TabPin3, symbol Regulator_Switching:LM2596S-3.3
- removed VR1: TPS561208DDCR, Package_TO_SOT_SMD:TSOT-23-6_HandSoldering, symbol TPS561208DDCR:TPS561208DDCR
- added C10, C9: 5pF, Capacitor_SMD:C_0603_1608Metric, symbol Device:C_Small
- added C11, C12, C16, C18: 0.1uF, Capacitor_SMD:C_0603_1608Metric, symbol Device:C
- added C13: 22uF, Capacitor_SMD:C_0603_1608Metric, symbol Device:C
- added C14: 33nF, Capacitor_SMD:C_0603_1608Metric, symbol Device:C
- added C15, C21: 1uF, Capacitor_SMD:C_0603_1608Metric, symbol Device:C
- added C17: 2.2nF, Capacitor_SMD:C_0603_1608Metric, symbol Device:C
- added C19, C20: 47pF, Capacitor_SMD:C_0603_1608Metric, symbol Device:C
- added C22: 60uF, Capacitor_SMD:C_0603_1608Metric, symbol Device:C
- added C23, C24, C25, C26, C27, C28: 0.1uF, Capacitor_SMD:C_0603_1608Metric, symbol Device:C_Small
- added D1: 45V16A1, Package_TO_SOT_THT:TO-220-2_Vertical, symbol Device:D_Schottky
- added D2: 18VWM29.2VC1, Diode_SMD:D_SOD-123, symbol Device:D_Zener
- added F1: MF-RHT1000, Fuse:Fuse_Bourns_MF-RHT1000, symbol Device:Polyfuse
- added H1, H2, H3, H4: MountingHole, MountingHole:MountingHole_2.7mm, symbol Mechanical:MountingHole
- added J10: Conn_02x20_Odd_Even, Connector_PinSocket_2.54mm:PinSocket_2x20_P2.54mm_Vertical, symbol Connector_Generic:Conn_02x20_Odd_Even
- added J11: Conn_01x04_Pin, Connector_PinHeader_2.54mm:PinHeader_1x04_P2.54mm_Vertical, symbol Connector:Conn_01x04_Pin
- added J12: Battery holes, 1984617(1):PHOENIX_1984617, symbol Connector_Generic:Conn_01x02
- added J13: USB_C_Receptacle, Connector_USB:USB_C_Receptacle_Amphenol_12401610E4-2A, symbol Connector:USB_C_Receptacle
- added R21: 100kR, Resistor_SMD:R_0603_1608Metric, symbol Device:R_Small_US
- added R22: 10R, Resistor_SMD:R_0603_1608Metric, symbol Device:R_US
- added R25, R26: 4.7kR, Resistor_SMD:R_0603_1608Metric, symbol Device:R_Small_US
- added R27: 20kR, Resistor_SMD:R_0603_1608Metric, symbol Device:R_US
- added R28: 110kR, Resistor_SMD:R_0603_1608Metric, symbol Device:R_US
- added R29: 15kR, Resistor_SMD:R_0603_1608Metric, symbol Device:R_US
- added R31, R32: 5.1kR, Resistor_SMD:R_0603_1608Metric, symbol Device:R_US
- added U6: STM32F091RCT6, Package_QFP:LQFP-64_10x10mm_P0.5mm, symbol STM32FO91RCT6:STM32F091RCT6
- added U7: INA226AQDGSRQ1, Package_SO:VSSOP-10_3x3mm_P0.5mm, symbol INA226AQDGSRQ1:INA226AQDGSRQ1
- added U8: AOZ6605PI-1, AOZ6605PI-1:SO8_EP1_AOS, symbol AOZ6605PI-1:AOZ6605PI-1
- added U9: MIC5219-3.3YMM, Package_SO:MSOP-8_3x3mm_P0.65mm, symbol Regulator_Linear:MIC5219-3.3YMM
- added Y1: CM7V-T1A-32.768kHz-7pF, Crystal:Crystal_SMD_3215-2Pin_3.2x1.5mm, symbol Device:Crystal_Small
- L2: value L -> 4.7uH; footprint Inductor_SMD:L_Chilisin_BMRA00050530 -> 74437377047:WE-LHMI_1335
- R23: value R_US -> 7.5mR; footprint Resistor_SMD:R_0603_1608Metric -> Resistor_SMD:R_2512_6332Metric
- R24: value R_US -> 10R
Connections:
- net +3V3: now also C12.2, C21.1, C23.1, C24.1, C25.1, C26.1, C27.1, C28.2, J11.4 (Pin_4), R21.2, R25.1, R26.1, U6.1 (VBAT), U6.13 (VDDA), U6.19 (VDD), U6.31 (VSS), U6.32 (VDD), U6.48 (VDDIO2), U6.63 (VSS), U6.64 (VDD), U9.3 (OUT); no longer L2.2
- net +5V: now also L2.2, C15.1, C20.1, C22.1, J10.2 (Pin_2), J10.4 (Pin_4), J13.A4 (VBUS), J13.A9 (VBUS), J13.B4 (VBUS), J13.B9 (VBUS), R28.2, U9.1 (EN), U9.2 (IN); no longer R23.1
- net GND: now also C10.1, C13.2, C14.1, C15.2, C16.2, C17.2, C19.2, C21.2, C22.2, C23.2, C24.2, C25.2, C26.2, C27.2, C28.1, C9.1, D2.2 (A), J10.14 (Pin_14), J10.20 (Pin_20), J10.25 (Pin_25), J10.30 (Pin_30), J10.34 (Pin_34), J10.39 (Pin_39), J10.6 (Pin_6), J10.9 (Pin_9), J11.1 (Pin_1), J12.1 (Pin_1), J13.A1 (GND), J13.A12 (GND), J13.B1 (GND), J13.B12 (GND), J13.S1 (SHIELD), R29.1, R31.2, R32.2, U6.12 (VSSA), U6.18 (VSS), U6.47 (VSS), U7.1 (A1), U7.2 (A0), U7.7 (GND), U8.4 (GND), U9.5 (GND), U9.6 (GND), U9.7 (GND), U9.8 (GND)
- net SPI1_MISO: now also U6.56 (PB4)
- net SPI1_MOSI: now also U6.57 (PB5)
- net SPI1_SCK: now also U6.21 (PA5)
- net UART1_RX: now also J10.8 (Pin_8), U6.59 (PB7)
- net UART1_TX: now also J10.10 (Pin_10), U6.58 (PB6)
- net UART2_RX: now also U6.17 (PA3)
- net UART2_TX: now also U6.16 (PA2)
- net at R24.1: now also C11.1; no longer R23.2
- net VBAT: now reaches R24.2
- net VBAT: now also R23.2, D1.1 (K), D2.1 (K)
- net at L2.1: now also C18.1, U8.EPAD (LX)
- new net: F1.1, J12.2 (Pin_2)
- new net: D1.2 (A), F1.2
- new net: C18.2, U8.5 (BST)
- new net: C20.2, R28.1, R29.2, U8.8 (FB)
- new net: C14.2, U8.1 (SS)
- new net: C16.1, U8.6 (VCC)
- new net: C19.1, R27.1, U8.7 (COMP)
- new net: C9.2, U6.3 (PC14-OSC32_IN), Y1.2
- new net: J13.A5 (CC1), R31.1
- new net: J13.B5 (CC2), R32.1
- new net: C12.1, U7.6 (VS)
- new net: C17.1, R27.2
- new net: C10.2, U6.4 (PC15-OSC32_OUT), Y1.1
- new net: R22.1, U7.8 (VBUS), U7.9 (IN-)
- new net: C11.2, U7.10 (IN+)
- new net BOOT0: J10.29 (Pin_29), U6.60 (PF11-BOOT0)
- new net I2C1_SCK: R25.2, U6.6 (PF1-OSC_OUT), U7.5 (SCL)
- new net I2C1_SDA: R26.2, U6.5 (PF0-OSC_IN), U7.4 (SDA)
- new net IMU_INT: U6.61 (PB8)
- new net IMU_nCS: U6.28 (PB2)
- new net M1_ENCA: U6.14 (PA0)
- new net M1_ENCB: U6.15 (PA1)
- new net M1_IN1_PWM: U6.41 (PA8)
- new net M1_IN2_PWM: U6.42 (PA9)
- new net M2_ENCA: U6.29 (PB10)
- new net M2_ENCB: U6.30 (PB11)
- new net M2_IN1_PWM: U6.43 (PA10)
- new net M2_IN2_PWM: U6.44 (PA11)
- new net NRST: J10.31 (Pin_31), R21.1, U6.7 (NRST)
- new net SERVO_PWM: U6.20 (PA4)
- new net SPREADER_MOTOR_EN: U6.37 (PC6)
- new net SWCLK: J11.2 (Pin_2), U6.49 (PA14)
- new net SWDIO: J11.3 (Pin_3), U6.46 (PA13)
- new net US1_ECHO: U6.22 (PA6)
- new net US1_TRIG: U6.8 (PC0)
- new net US2_ECHO: U6.23 (PA7)
- new net US2_TRIG: U6.9 (PC1)
- new net US3_ECHO: U6.26 (PB0)
- new net US3_TRIG: U6.10 (PC2)
- new net US4_ECHO: U6.27 (PB1)
- new net US4_TRIG: U6.11 (PC3)
- new net VBAT_LOAD: C13.1, R22.2, R23.1, U8.2 (EN), U8.3 (VIN)
- no-connect marks 0 -> 60
Other:
- note removed: "12C1_SCL/TIM16_CH1/FTf"
- note removed: "12C1_SCL/USART1_TX/FTf"
- note removed: "12C1_SDA/TIM17_CH1/FTf"
- note removed: "12C1_SDA/USART1_RX/FTf"
- note removed: "12C2_SCL/USART3_TX/TIM2_CH3/FT"
- note removed: "12C2_SDA/USART3_RX/TIM2_CH4/FT"
- note removed: "ADC_IN8/TIM3_CH3/TTa"
- note removed: "ADC_IN9/TIM3_CH4/TTa"
- note removed: "FT"
- note removed: "FT/SPI1_NSS/USART2_RX"
- note removed: "FT/SWCLK/USART2_TX"
- note removed: "FT/SWDIO"
- note removed: "FT/TIM1_CH1"
- note removed: "FT/TIM1_CH2/USART1_TX"
- note removed: "FT/TIM1_CH3/USART1_RX"
- note removed: "Notes: FT and FTf are 3v TIM2 is used for SYSTICK SW Debug is on A13 and A14"
- note removed: "OSC32_IN/TC"
- note removed: "OSC32_OUT/TC"
- note removed: "OSC_IN/FT"
- note removed: "OSC_OUT/FT"
- note removed: "SPI1_SCK/TIM2_CH2/FT"
- note removed: "SPI2_MISO/I2C2_SDA/FTf"
- note removed: "SPI2_MOSI/FT"
- note removed: "SPI2_NSS/FT"
- note removed: "SPI2_SCK/I2C2_SCL/FTf"
- note removed: "SPI_MISO/TIM3_CH1/FT"
- note removed: "SPI_MOSI/TIM3_CH2/FT"
- note removed: "TTa/SPI1_SCK/ADC_IN5"
- note removed: "TTa/TIM14_CH1/SPI1_NSS/ADC_IN4"
- note removed: "TTa/TIM2_CH2/USART4_RX/ADC_IN1"
- note removed: "TTa/TIM2_CH3/USART2_TX/ADC_IN2"
- note removed: "TTa/TIM2_CH4/USART2_RX/ADC_IN3"
- note removed: "TTa/TIM3_CH1/SPI1_MISO/ADC_IN6"
- note removed: "TTa/TIM3_CH2/SPI_MOSI/ADC_IN7"
- note removed: "TTa/USART4_TX/ADC_IN0"
- note removed: "WKUP2/TC"
