File: MotroControl.kicad_sch (KiCad schematic)
At the start: 9 parts, among them M1 Motor_DC, M2 Motor_DC, M3 Motor_Servo, M4 Motor_DC, Q6 NMOS, U6 L298HN

Commit message: rev 1
Parts:
- removed M1, M2, M4: Motor_DC, Connector_PinHeader_1.27mm:PinHeader_1x02_P1.27mm_Vertical, symbol Motor:Motor_DC
- removed M3: Motor_Servo, Connector_PinHeader_2.54mm:PinHeader_1x03_P2.54mm_Vertical, symbol Motor:Motor_Servo
- removed Q6: NMOS, Package_TO_SOT_SMD:Infineon_PG-HSOF-8-1, symbol Simulation_SPICE:NMOS
- removed R21: 100KΩ, Resistor_SMD:R_0603_1608Metric, symbol Device:R_US
- removed U6: L298HN, Package_TO_SOT_THT:TO-220-15_P2.54x2.54mm_StaggerOdd_Lead5.84mm_TabDown, symbol Driver_Motor:L298HN
- added J2, J3, J6, J8: Conn_01x04, Connector_PinHeader_2.54mm:PinHeader_1x04_P2.54mm_Vertical, symbol Connector_Generic:Conn_01x04
- added J4, J5: Conn_01x06, Connector_JST:JST_PH_B6B-PH-K_1x06_P2.00mm_Vertical, symbol Connector_Generic:Conn_01x06
- added J7: Conn_01x03_Pin, Connector_PinHeader_2.54mm:PinHeader_1x03_P2.54mm_Vertical, symbol Connector:Conn_01x03_Pin
- added J9: Conn_01x02, 1984617(1):PHOENIX_1984617, symbol Connector_Generic:Conn_01x02
- added Q10: DMP3013SFV, Package_SON:Diodes_PowerDI3333-8, symbol Transistor_FET:DMP3013SFV
- added Q11, Q6, Q7, Q8, Q9: BSS138, Package_TO_SOT_SMD:SOT-23, symbol Transistor_FET:DMN2040U
- added R10, R11, R12, R13, R14, R15, R16, R17: 10kR, Resistor_SMD:R_0603_1608Metric, symbol Device:R_Small_US
- added R18: 100R, Resistor_SMD:R_0603_1608Metric, symbol Device:R_US
- added U5: L298HN, Package_TO_SOT_THT:TO-220-15_P2.54x2.54mm_StaggerOdd_Lead5.84mm_TabDown, symbol Driver_Motor:L298HN
- R19: value 100Ω -> 10kR
- R20: value 100Ω -> 50kR
Connections:
- net +5V: now also J2.1 (Pin_1), J3.1 (Pin_1), J6.1 (Pin_1), J7.2 (Pin_2), J8.1 (Pin_1), Q6.1 (G), Q7.1 (G), Q8.1 (G), Q9.1 (G), R10.2, R11.2, R12.2, R13.2, U5.11 (EnB), U5.6 (EnA), U5.9 (Vss)
- net GND: now also J2.4 (Pin_4), J3.4 (Pin_4), J4.5 (Pin_5), J5.5 (Pin_5), J6.4 (Pin_4), J7.3 (Pin_3), J8.4 (Pin_4), J9.2 (Pin_2), Q11.2 (S), U5.1 (SENSE_A), U5.15 (SENSE_B), U5.8 (GND)
- net at R19.2: now also R20.2, Q10.4 (G)
- net B13 renamed VBAT_LOAD
- net VBAT_LOAD: now also Q10.1 (S), Q10.2 (S), Q10.3 (S), U5.4 (Vs)
- net B14: no longer names the net of R19.1
- net B14: now also Q11.3 (D)
- new net: J7.1 (Pin_1), R18.2
- new net: J9.1 (Pin_1), Q10.5 (D)
- new net +3V3: J4.2 (Pin_2), J5.2 (Pin_2), R14.2, R15.2, R16.2, R17.2
- new net ECHO1: J2.3 (Pin_3), Q9.2 (S), R13.1
- new net ECHO2: J3.3 (Pin_3), Q7.2 (S), R11.1
- new net ECHO3: J6.3 (Pin_3), Q8.2 (S), R12.1
- new net ECHO4: J8.3 (Pin_3), Q6.2 (S), R10.1
- new net M1+: J4.1 (Pin_1), U5.2 (OUT1)
- new net M1-: J4.6 (Pin_6), U5.3 (OUT2)
- new net M1_ENCA: J4.3 (Pin_3)
- new net M1_ENCB: J4.4 (Pin_4)
- new net M1_IN1_PWM: U5.5 (IN1)
- new net M1_IN2_PWM: U5.7 (IN2)
- new net M2+: J5.1 (Pin_1), U5.13 (OUT3)
- new net M2-: J5.6 (Pin_6), U5.14 (OUT4)
- new net M2_ENCA: J5.3 (Pin_3)
- new net M2_ENCB: J5.4 (Pin_4)
- new net M2_IN1_PWM: U5.10 (IN3)
- new net M2_IN2_PWM: U5.12 (IN4)
- new net SERVO_PWM: R18.1
- new net SPREADER_MOTOR_EN: Q11.1 (G)
- new net US1_ECHO: Q9.3 (D), R17.1
- new net US1_TRIG: J2.2 (Pin_2)
- new net US2_ECHO: Q7.3 (D), R15.1
- new net US2_TRIG: J3.2 (Pin_2)
- new net US3_ECHO: Q8.3 (D), R16.1
- new net US3_TRIG: J6.2 (Pin_2)
- new net US4_ECHO: Q6.3 (D), R14.1
- new net US4_TRIG: J8.2 (Pin_2)
Other:
- note removed: "Motor Control"
